File: MainBoard/DS7A-2.kicad_pcb (KiCad board)
At the start: 2 copper layers, 165 x 172.5 mm, 93 parts, among them CON1 To FDD, J1 Barrel_Jack_Switch, J2 DB25_Receptacle_MountingHoles, Q1 BC846A SMD, Q2 2N3904 THT DNP, U10 74LS244, U4 27512

Commit message: Add files via upload
Other:
- outline, holes or cut-outs redrawn
- board text removed: "230 Ohm"
Changed lines of the file:
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@@
 	)
 	(gr_circle
-		(center 285 93.2)
-		(end 286.500033 93.2)
+		(center 286.3 93.2)
+		(end 287.800033 93.2)
 		(stroke
 			(width 0.002)
@@
 	)
 	(gr_circle
-		(center 285 213.2)
-		(end 286.500033 213.2)
+		(center 286.6 213)
+		(end 288.100033 213)
 		(stroke
 			(width 0.002)
@@
 		)
 	)
-	(gr_text "230 Ohm"
+	(gr_text "220 Ohm"
 		(at 255.8 216.18 0)
 		(layer "F.SilkS")
@@
 	)
 	(via
-		(at 287.5 95)
+		(at 282.5 95)
 		(size 0.6)
 		(drill 0.3)
