File: MainBoard/DS7A-2.kicad_pcb (KiCad board)
At the start: 2 copper layers, 165 x 172.5 mm, 93 parts, among them CON1 To FDD, J1 Barrel_Jack_Switch, J2 DB25_Receptacle_MountingHoles, Q1 BC846A SMD, Q2 2N3904 THT DNP, U10 74LS244, U4 27512

Commit message: Add files via upload
Parts:
- REG1: footprint Package_TO_SOT_THT:TO-220-3_Horizontal_TabDown -> Package_TO_SOT_THT:TO-220-3_Vertical
Connections:
- U9 pad 112: unconnected-(U9-FDC_TC-Pad112) -> /TC
Routing:
- net /TC: track 0.00 -> 59.0 mm, vias 0 -> 2
- net /GND: track 1092.9 -> 1085.9 mm
- net /~{CS}.FDC: track 76.7 -> 76.0 mm
