File: MainBoard/DS7A-2.kicad_sch (KiCad schematic)
At the start: 93 parts, among them CON1 To FDD, J1 Barrel_Jack_Switch, J2 DB25_Receptacle_MountingHoles, Q1 BC846A SMD, Q2 2N3904 THT DNP, U10 74LS244, U4 27512

Commit message: Add files via upload
Parts:
- CN1, CN2, U12, U14, U2, U3, U5, U6, U9: value ~ -> (none)
Connections:
- net TC: now also U9.112 (FDC_TC)
